Commit message: Parameterize thruster model type

File: rov_description/models/t200_thruster.xacro (robot description, xacro)
@@ -1,4 +1,4 @@
 <robot xmlns:xacro="http://www.ros.org/wiki/xacro">
-    <xacro:macro name="t200_thruster" params="name pose">
+    <xacro:macro name="t200_thruster" params="name pose prop_type">
         <link name="${name}">
             <pose>${pose}</pose>
@@ -7,5 +7,5 @@
                 <geometry>
                     <mesh>
-                        <uri>model://meshes/t200-cw-prop.dae</uri>
+                        <uri>model://meshes/t200-${prop_type}-prop.dae</uri>
                     </mesh>
                 </geometry>
