Commit message: Camera work now

File: rov_description/models/camera.xacro (robot description, xacro)
@@ -1,49 +1,56 @@
 <?xml version="1.0" encoding="UTF-8"?>
 <robot xmlns:xacro="http://www.ros.org/wiki/xacro">
-    <xacro:macro name="lowlight_cam" params="name parent xyz rpy">
-        <!-- <model name="camera"> -->
-        <!-- <pose>4 0 1.0 0 0.0 3.14</pose> -->
-        <joint name="${name}_joint" type="fixed">
-            <!-- <origin xyz="0.305 0 0.08" rpy="0 0 0" /> -->
-            <parent>${parent}</parent>
-            <child>${name}_link</child>
-        </joint>
-        <link name="${name}_link">
-            <pose>${xyz} ${rpy}</pose>
-            <visual name="${name}_link_visual">
-                <geometry>
-                    <box>
-                        <size>0.010 0.03 0.03</size>
-                    </box>
-                </geometry>
-                <!-- <material name="red" /> -->
-            </visual>
-        </link>
-        <!-- Dummy link for converting from standard ROS orientation to standard optical -->
-        <!-- Standard ROS:     (x-forward, y-left, z-up) -->
-        <!-- Standard Optical: (x-right  , y-down, z-forward)-->
-        <joint name="${name}_optical_joint" type="fixed">
-            <!-- <origin xyz="0 0 0" rpy="${pi/2} 0 ${pi/2}" /> -->
-            <parent>${name}_link</parent>
-            <child>${name}_link_optical</child>
-        </joint>
-        <link name="${name}_link_optical">
-            <sensor name="${name}" type="camera">
-                <camera>
-                    <horizontal_fov>${80 * pi/180}</horizontal_fov>n <image>
-                        <width>1920</width>
-                        <height>1080</height>
-                    </image>
-                    <clip>
-                        <near>0.1</near>
-                        <far>100</far>
-                    </clip>
-                </camera>
-                <topic>camera_topic</topic>
-                <always_on>1</always_on>
-                <update_rate>30</update_rate>
-                <visualize>true</visualize>
-            </sensor>
-        </link>
-    </xacro:macro>
+  <xacro:macro name="lowlight_cam" params="name parent xyz rpy">
+    <model name="camera">
+    <!-- <pose>4 0 1.0 0 0.0 3.14</pose> -->
+    <joint name="${name}_joint" type="fixed">
+      <!-- <origin xyz="0.305 0 0.08" rpy="0 0 0" /> -->
+      <parent>${parent}</parent>
+      <child>${name}_link</child>
+    </joint>
+    <link name="${name}_link">
+      <pose>${xyz} ${rpy}</pose>
+      <visual name="${name}_link_visual">
+        <geometry>
+          <box>
+            <size>0.010 0.03 0.03</size>
+          </box>
+        </geometry>
+        <!-- <material name="red" /> -->
+      </visual>
+    </link>
+    <!-- Dummy link for converting from standard ROS orientation to standard optical -->
+    <!-- Standard ROS:     (x-forward, y-left, z-up) -->
+    <!-- Standard Optical: (x-right  , y-down, z-forward)-->
+    <joint name="${name}_optical_joint" type="fixed">
+      <!-- <origin xyz="0 0 0" rpy="${pi/2} 0 ${pi/2}" /> -->
+      <parent>${name}_link</parent>
+      <child>${name}_link_optical</child>
+    </joint>
+    <link name="${name}_link_optical">
+      <sensor name="${name}" type="camera">
+        <camera>
+          <horizontal_fov>${80 * pi/180}</horizontal_fov>
+          <image>
+            <width>1920</width>
+            <height>1080</height>
+          </image>
+          <clip>
+            <near>0.1</near>
+            <far>100</far>
+          </clip>
+        </camera>
+        <topic>camera_topic</topic>
+        <always_on>1</always_on>
+        <update_rate>30</update_rate>
+        <visualize>true</visualize>
+      </sensor>
+    </link>
+    </model>
+    <joint name="${name}_joint" type="fixed">
+      <!-- <origin xyz="0.305 0 0.08" rpy="0 0 0" /> -->
+      <parent>${parent}</parent>
+      <child>camera::${name}_link</child>
+    </joint>
+  </xacro:macro>
 </robot>
